File: cm5io/PCIe-M2.kicad_sch (KiCad schematic)
At the start: 24 parts, among them J4 Bus_M.2_Socket_M, M1 M.2 Screw, M2 M.2 Solder Nut, M3 M.2 Solder Nut, M4 M.2 Solder Nut, M5 M.2 Solder Nut, U7 ASEK-32.768KHZ-L-R-T, U8 AP3441SHE-7B

Commit message: [cm5io] remove USB-C and NVMe connectors, clean up routing
Parts:
- removed C10, C19: 100n, Capacitor_SMD:C_0402_1005Metric, symbol Device:C
- removed C11: 4.7nF, Capacitor_SMD:C_0402_1005Metric, symbol Device:C
- removed C14, C15, C16, C17, C4, C6: 10u, Capacitor_SMD:C_0805_2012Metric, symbol Device:C
- removed D3: LED Green, LED_SMD:LED_0603_1608Metric, symbol Device:LED
- removed J4: Bus_M.2_Socket_M, CM5IO:M.2 M Key socket, symbol CM5IO:Bus_M.2_Socket_M
- removed L1: 2.2uH, CM5IO:L_Bourns_SRP5030CC, symbol Device:L
- removed M1: M.2 Screw, symbol CM5IO:M.2_Screw
- removed M2, M3, M4, M5: M.2 Solder Nut, symbol CM5IO:SolderNut
- removed R14: 100K 1%, Resistor_SMD:R_0402_1005Metric, symbol Device:R
- removed R15: 10K 1%, Resistor_SMD:R_0402_1005Metric, symbol Device:R
- removed R16: 2.2K 1%, Resistor_SMD:R_0402_1005Metric, symbol Device:R
- removed R17: 1k, Resistor_SMD:R_0402_1005Metric, symbol Device:R
- removed TP1: TestPoint, TestPoint:TestPoint_Pad_2.0x2.0mm, symbol Connector:TestPoint
- removed U7: ASEK-32.768KHZ-L-R-T, Crystal:Crystal_SMD_3225-4Pin_3.2x2.5mm, symbol CM5IO:ASEK-32.768KHZ-L-R-T
- removed U8: AP3441SHE-7B, Package_DFN_QFN:DFN-8-1EP_2x2mm_P0.5mm_EP1.05x1.75mm, symbol CM5IO:AP3441SHE-7B
Connections:
- no-connect marks 15 -> 0
Other:
- note removed: "Activity LED"
